File: sensor_machine.kicad_pcb (KiCad board)
At the start: 2 copper layers, 83.1 x 61.6 mm, 24 parts, among them J1 Barrel_Jack, J11 Screw_Terminal_01x02, J2 Barrel_Jack_Switch, J3 Screw_Terminal_01x02, J4 Screw_Terminal_01x02, J5 Screw_Terminal_01x02, J7 Screw_Terminal_01x02, J8 Screw_Terminal_01x02, J9 Screw_Terminal_01x01, U1 ard_UNO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

Commit message: modificaciones PCB
Parts:
- removed ?: Screw_Terminal_01x01, Connector_Wire:SolderWirePad_1x01_Drill0.8mm
- removed J1: Barrel_Jack, Connector_BarrelJack:BarrelJack_Horizontal
- added J6: Screw_Terminal_01x02, TerminalBlock:TerminalBlock_Altech_AK300-2_P5.00mm, F.Cu at (134.9, 119.0)
- J7: value Screw_Terminal_01x02 -> Screw_Terminal_01x01; footprint TerminalBlock:TerminalBlock_Altech_AK300-2_P5.00mm -> Connectors:Pin_d1.0mm_L10.0mm
- J9: footprint Connector_Wire:SolderWirePad_1x01_Drill0.8mm -> Connectors:Pin_d1.0mm_L10.0mm
- moved J7 41.9 mm to (171.0, 122.9)
- moved J9 2.93 mm to (143.0, 122.8)
- moved D3 2.55 mm to (163.6, 80.4)
- moved J2 1.55 mm to (142.4, 79.5)
- moved C4 1.29 mm to (148.8, 103.6)
Connections:
- J2 pad 2: Net-(J1-Pad1) -> /Vin
- J4 pad 1: Net-(J4-Pad1) -> /Vin
- J7 pad 1: Net-(J7-Pad1) -> /A5
- J9 pad 1: Net-(J7-Pad1) -> /A5'
- R3 pad 1: Net-(J4-Pad1) -> /Vin
- U1 pad 14: Net-(J6-Pad1) -> /A5
Routing:
- net /Vin: track 0.00 -> 139.7 mm
- net Net-(J1-Pad1): track 74.9 -> 0.00 mm
- net Net-(J4-Pad1): track 22.7 -> 0.00 mm
- net Net-(J7-Pad1): track 15.1 -> 0.00 mm
- net /A5': track 0.00 -> 12.5 mm
- net /5v: track 65.3 -> 53.0 mm
- net /A5: track 0.00 -> 5.73 mm
- net Net-(J6-Pad1): track 3.88 -> 0.00 mm
- net +12V: track 52.7 -> 49.8 mm
- net /A3: track 30.0 -> 28.9 mm
- net +7.5V: track 69.5 -> 70.0 mm
Other:
- board size 83.1 x 61.6 mm -> 83.1 x 61.8 mm
- board text added: "A5"
- board text removed: "A0"
