File: sensor_machine.sch (KiCad schematic (older format))
At the start: 19 parts, among them J1 Barrel_Jack, J2 Barrel_Jack_Switch, J3 Screw_Terminal_01x02, J4 Screw_Terminal_01x02, J5 Screw_Terminal_01x02, J6 Screw_Terminal_01x02, U2 LM317_3PinPackage

Commit message: modificaciones pcb con arduino UNO
Parts:
- removed J6: Screw_Terminal_01x02, TerminalBlock:TerminalBlock_Altech_AK300-2_P5.00mm, symbol Connector:Screw_Terminal_01x02
- added J11, J3, J7: Screw_Terminal_01x02, TerminalBlock:TerminalBlock_Altech_AK300-2_P5.00mm, symbol Connector:Screw_Terminal_01x02
- added U1: ard_UNO, ard_UNO:arduino_UNO, symbol arduino_UNO:ard_UNO
- renumbered J3 to J8
Connections:
- net GND: now also J4.2 (Pin_2), J11.2 (Pin_2), J3.2 (Pin_2), J7.2 (Pin_2), U1.29 (GND), U1.6 (GND), U1.7 (GND); no longer J4.1 (Pin_1)
- net at D3.1 (K): now also J3.1 (Pin_1); no longer J8.1 (Pin_1)
- net at D4.1 (K): now also J5.1 (Pin_1)
- net at R3.1: now also J4.1 (Pin_1); no longer J4.2 (Pin_2)
- net A3: now reaches C1.1, R3.2, R5.1
- net A3: now also U1.12 (A3); no longer J5.1 (Pin_1)
- new net A5: J7.1 (Pin_1), U1.14 (A5)
- new net D4: J11.1 (Pin_1), U1.19 (4)
- new net D6: J8.1 (Pin_1), U1.21 (6)
- no-connect marks 0 -> 25
Other:
- moved on the sheet: C1, C2, C4, D1, D2, D3, D4, J1, J2, J8, R1, R2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

Commit message: reconfiguracion pcb
Parts:
- added J6, J9: Screw_Terminal_01x01, Connector_Wire:SolderWirePad_1x01_Drill0.8mm, symbol Connector:Screw_Terminal_01x01
- R2: value 120 -> 1200
Connections:
- net at D3.1 (K): no longer J3.1 (Pin_1)
- net 5v: now reaches U1.5 (5V)
- net 5v: now also J3.1 (Pin_1)
- net +9V renamed +7.5V
- net A5: no longer names the net of J7.1 (Pin_1)
- net A5: now also J9.1 (Pin_1); no longer U1.14 (A5)
- new net: J6.1 (Pin_1), U1.14 (A5)
- no-connect marks 25 -> 24
Other:
- moved on the sheet: D3
Changed lines of the file:
@@
 P 4750 4000
 F 0 "R2" H 4820 4046 50  0000 L CNN
-F 1 "120" H 4820 3955 50  0000 L CNN
+F 1 "1200" H 4820 3955 50  0000 L CNN
 F 2 "Resistor_THT:R_Axial_DIN0207_L6.3mm_D2.5mm_P10.16mm_Horizontal" V 4680 4000 50  0001 C CNN
 F 3 "~" H 4750 4000 50  0001 C CNN
@@
 Wire Wire Line
 	5150 3200 5250 3200
-$Comp
-L power:+9V #PWR011
-U 1 1 5C808D41
-P 5400 3200
-F 0 "#PWR011" H 5400 3050 50  0001 C CNN
-F 1 "+9V" H 5415 3373 50  0000 C CNN
-F 2 "" H 5400 3200 50  0001 C CNN
-F 3 "" H 5400 3200 50  0001 C CNN
-	1    5400 3200
-	1    0    0    -1
-$EndComp
 Wire Wire Line
 	5400 3200 5900 3200
@@
 L Diode:1N4001 D3
 U 1 1 5D4C4754
-P 5100 2300
-F 0 "D3" H 5100 2084 50  0000 C CNN
-F 1 "1N4001" H 5100 2175 50  0000 C CNN
-F 2 "Diode_THT:D_DO-41_SOD81_P10.16mm_Horizontal" H 5100 2125 50  0001 C CNN
-F 3 "http://www.vishay.com/docs/88503/1n4001.pdf" H 5100 2300 50  0001 C CNN
-	1    5100 2300
+P 4800 2300
+F 0 "D3" H 4800 2084 50  0000 C CNN
+F 1 "1N4001" H 4800 2175 50  0000 C CNN
+F 2 "Diode_THT:D_DO-41_SOD81_P10.16mm_Horizontal" H 4800 2125 50  0001 C CNN
+F 3 "http://www.vishay.com/docs/88503/1n4001.pdf" H 4800 2300 50  0001 C CNN
+	1    4800 2300
 	-1   0    0    1
 $EndComp
 Wire Wire Line
-	4950 2300 4000 2300
+	4650 2300 4000 2300
 $Comp
 L Device:R R3
@@
 Wire Wire Line
 	4300 3550 4300 3650
-Wire Wire Line
-	6450 3200 6300 3200
 $Comp
 L power:GND #PWR0101
@@
 Wire Wire Line
 	7650 3850 7500 3850
-Text Label 7500 3850 2    50   ~ 0
-A5
 Wire Wire Line
 	7650 3650 7500 3650
@@
 Text Label 8700 3450 0    50   ~ 0
 D4
-Wire Wire Line
-	5400 2300 5250 2300
 $Comp
 L Connector:Screw_Terminal_01x02 J3
@@
 	1    0    0    -1
 $EndComp
-Text Label 7550 4700 0    50   ~ 0
-A5
 $Comp
 L Connector:Screw_Terminal_01x02 J4
@@
 NoConn ~ 7650 2700
 NoConn ~ 7650 2800
-NoConn ~ 7650 2900
 NoConn ~ 7650 3350
 NoConn ~ 7650 3450
@@
 	1    0    0    -1
 $EndComp
+Text Label 5300 2300 0    50   ~ 0
+5v
+Text Label 7650 2900 0    50   ~ 0
+5v
+Wire Wire Line
+	5400 2300 5300 2300
+Wire Wire Line
+	6300 3200 6450 3200
+$Comp
+L power:+7.5V #PWR0111
+U 1 1 5D707C72
+P 5400 3200
+F 0 "#PWR0111" H 5400 3050 50  0001 C CNN
+F 1 "+7.5V" H 5415 3373 50  0000 C CNN
+F 2 "" H 5400 3200 50  0001 C CNN
+F 3 "" H 5400 3200 50  0001 C CNN
+	1    5400 3200
+	1    0    0    -1
+$EndComp
+$Comp
+L Connector:Screw_Terminal_01x01 J9
+U 1 1 5D75DCB4
+P 7350 4700
+F 0 "J9" H 7270 4475 50  0000 C CNN
+F 1 "Screw_Terminal_01x01" H 7270 4566 50  0000 C CNN
+F 2 "Connector_Wire:SolderWirePad_1x01_Drill0.8mm" H 7350 4700 50  0001 C CNN
+F 3 "~" H 7350 4700 50  0001 C CNN
+	1    7350 4700
+	-1   0    0    1
+$EndComp
+$Comp
+L Connector:Screw_Terminal_01x01 J6
+U 1 1 5D75DE44
+P 7300 3850
+F 0 "J6" H 7220 3625 50  0000 C CNN
+F 1 "Screw_Terminal_01x01" H 7220 3716 50  0000 C CNN
+F 2 "Connector_Wire:SolderWirePad_1x01_Drill0.8mm" H 7300 3850 50  0001 C CNN
+F 3 "~" H 7300 3850 50  0001 C CNN
+	1    7300 3850
+	-1   0    0    1
+$EndComp
 $EndSCHEMATC

Commit message: modificaciones PCB
Parts:
- removed J6: Screw_Terminal_01x01, Connector_Wire:SolderWirePad_1x01_Drill0.8mm, symbol Connector:Screw_Terminal_01x01
- removed J7: Screw_Terminal_01x02, TerminalBlock:TerminalBlock_Altech_AK300-2_P5.00mm, symbol Connector:Screw_Terminal_01x02
- added J6: Screw_Terminal_01x02, TerminalBlock:TerminalBlock_Altech_AK300-2_P5.00mm, symbol Connector:Screw_Terminal_01x02
- added J7: Screw_Terminal_01x01, Connectors:Pin_d1.0mm_L10.0mm, symbol Connector:Screw_Terminal_01x01
- J9: footprint Connector_Wire:SolderWirePad_1x01_Drill0.8mm -> Connectors:Pin_d1.0mm_L10.0mm
- U1: footprint ard_UNO:arduino_UNO -> ard_UNO:Arduino_UNO_R3_WithMountingHoles_handsoldering
Connections:
- net GND: now also J6.2 (Pin_2)
- net Vin: now reaches J1.1, J2.2
- net Vin: now also J4.1 (Pin_1), R3.1
- net A5': now reaches J9.1 (Pin_1)
- net A5': now also J6.1 (Pin_1)
- net A5: now reaches U1.14 (A5)
- net A5: now also J7.1 (Pin_1)
Changed lines of the file:
@@
 	5400 3600 5400 3550
 Wire Wire Line
-	3050 2750 3500 2750
+	3050 2750 3250 2750
 $Comp
 L Diode:1N4001 D1
@@
 A3
 Wire Wire Line
-	7650 3850 7500 3850
-Wire Wire Line
 	7650 3650 7500 3650
 Text Label 7500 3650 2    50   ~ 0
@@
 F 3 "~" H 5600 2300 50  0001 C CNN
 	1    5600 2300
-	1    0    0    -1
-$EndComp
-$Comp
-L power:GND #PWR0105
-U 1 1 5D6D470C
-P 7700 4800
-F 0 "#PWR0105" H 7700 4550 50  0001 C CNN
-F 1 "GND" H 7705 4627 50  0000 C CNN
-F 2 "" H 7700 4800 50  0001 C CNN
-F 3 "" H 7700 4800 50  0001 C CNN
-	1    7700 4800
-	1    0    0    -1
-$EndComp
-Wire Wire Line
-	7700 4700 7550 4700
-$Comp
-L Connector:Screw_Terminal_01x02 J7
-U 1 1 5D6D4713
-P 7900 4700
-F 0 "J7" H 7980 4692 50  0000 L CNN
-F 1 "Screw_Terminal_01x02" H 7980 4601 50  0000 L CNN
-F 2 "TerminalBlock:TerminalBlock_Altech_AK300-2_P5.00mm" H 7900 4700 50  0001 C CNN
-F 3 "~" H 7900 4700 50  0001 C CNN
-	1    7900 4700
 	1    0    0    -1
 $EndComp
@@
 F 0 "U1" H 8100 3175 50  0000 C CNN
 F 1 "ard_UNO" H 8100 3084 50  0000 C CNN
-F 2 "ard_UNO:arduino_UNO" H 8150 2500 50  0001 C CNN
+F 2 "ard_UNO:Arduino_UNO_R3_WithMountingHoles_handsoldering" H 8150 2500 50  0001 C CNN
 F 3 "" H 8150 2500 50  0001 C CNN
 	1    8100 2500
@@
 	1    0    0    -1
 $EndComp
+Wire Wire Line
+	3250 2750 3250 2950
+Wire Wire Line
+	3250 2950 3350 2950
+Connection ~ 3250 2750
+Wire Wire Line
+	3250 2750 3500 2750
+Text Label 3350 2950 0    50   ~ 0
+Vin
+Text Label 5600 4550 0    50   ~ 0
+Vin
+Wire Wire Line
+	5600 4550 5300 4550
+Connection ~ 5300 4550
+Text Label 7550 4600 0    50   ~ 0
+A5'
+$Comp
+L Connector:Screw_Terminal_01x02 J6
+U 1 1 5DEB5F66
+P 7900 4600
+F 0 "J6" H 7980 4592 50  0000 L CNN
+F 1 "Screw_Terminal_01x02" H 7980 4501 50  0000 L CNN
+F 2 "TerminalBlock:TerminalBlock_Altech_AK300-2_P5.00mm" H 7900 4600 50  0001 C CNN
+F 3 "~" H 7900 4600 50  0001 C CNN
+	1    7900 4600
+	1    0    0    -1
+$EndComp
+Wire Wire Line
+	7700 4600 7550 4600
+Wire Wire Line
+	7700 4700 7700 4750
+$Comp
+L power:GND #PWR0105
+U 1 1 5DEB5F6F
+P 7700 4750
+F 0 "#PWR0105" H 7700 4500 50  0001 C CNN
+F 1 "GND" H 7705 4577 50  0000 C CNN
+F 2 "" H 7700 4750 50  0001 C CNN
+F 3 "" H 7700 4750 50  0001 C CNN
+	1    7700 4750
+	1    0    0    -1
+$EndComp
+Wire Wire Line
+	7650 3850 7500 3850
+Text Label 7500 3850 0    50   ~ 0
+A5
 $Comp
 L Connector:Screw_Terminal_01x01 J9
-U 1 1 5D75DCB4
-P 7350 4700
-F 0 "J9" H 7270 4475 50  0000 C CNN
-F 1 "Screw_Terminal_01x01" H 7270 4566 50  0000 C CNN
-F 2 "Connector_Wire:SolderWirePad_1x01_Drill0.8mm" H 7350 4700 50  0001 C CNN
-F 3 "~" H 7350 4700 50  0001 C CNN
-	1    7350 4700
+U 1 1 5DEBA7A8
+P 7350 4600
+F 0 "J9" H 7270 4375 50  0000 C CNN
+F 1 "Screw_Terminal_01x01" H 7270 4466 50  0000 C CNN
+F 2 "Connectors:Pin_d1.0mm_L10.0mm" H 7350 4600 50  0001 C CNN
+F 3 "~" H 7350 4600 50  0001 C CNN
+	1    7350 4600
 	-1   0    0    1
 $EndComp
 $Comp
-L Connector:Screw_Terminal_01x01 J6
-U 1 1 5D75DE44
+L Connector:Screw_Terminal_01x01 J7
+U 1 1 5DEBA869
 P 7300 3850
-F 0 "J6" H 7220 3625 50  0000 C CNN
-F 1 "Screw_Terminal_01x01" H 7220 3716 50  0000 C CNN
-F 2 "Connector_Wire:SolderWirePad_1x01_Drill0.8mm" H 7300 3850 50  0001 C CNN
+F 0 "J7" H 7300 3650 50  0000 C CNN
+F 1 "Screw_Terminal_01x01" H 7300 3750 50  0000 C CNN
+F 2 "Connectors:Pin_d1.0mm_L10.0mm" H 7300 3850 50  0001 R CNN
 F 3 "~" H 7300 3850 50  0001 C CNN
 	1    7300 3850
-	-1   0    0    1
+	-1   0    0    -1
 $EndComp
 $EndSCHEMATC
